Commit message: feat(m2.5): implement hackathon visualization, deterministic camera, demo scene, and fleet dashboard

File: src/amr_fleet_description/urdf/amr.urdf.xacro (robot description, xacro)
@@ -17,4 +17,5 @@
   <!-- Instantiate components -->
   <xacro:amr_core
+    robot_name="$(arg robot_name)"
     prefix="$(arg prefix)"
     chassis_length="$(arg chassis_length)"

File: src/amr_fleet_description/urdf/amr_core.xacro (robot description, xacro)
@@ -3,4 +3,5 @@
   <xacro:macro name="amr_core" params="
     prefix
+    robot_name:=amr_0
     chassis_length:=0.65
     chassis_width:=0.45
@@ -23,17 +24,60 @@
     </joint>
     <link name="${prefix}base_link">
-      <visual>
+      <!-- 1. Lower Industrial Chassis Base -->
+      <visual name="chassis_lower">
+        <origin xyz="0 0 ${chassis_height * 0.35}" rpy="0 0 0"/>
+        <geometry>
+          <box size="${chassis_length} ${chassis_width} ${chassis_height * 0.70}"/>
+        </geometry>
+        <material name="amr_chassis_dark"/>
+      </visual>
+      <!-- 2. Upper Protective Shell & Deck (Safety Orange) -->
+      <visual name="chassis_upper_shell">
+        <origin xyz="0 0 ${chassis_height * 0.82}" rpy="0 0 0"/>
+        <geometry>
+          <box size="${chassis_length * 0.96} ${chassis_width * 0.94} ${chassis_height * 0.28}"/>
+        </geometry>
+        <material name="amr_safety_orange"/>
+      </visual>
+      <!-- 3. Identification Badge Base (Dark Contrast Plate) -->
+      <visual name="id_badge_base">
+        <origin xyz="0 0 ${chassis_height + 0.003}" rpy="0 0 0"/>
+        <geometry>
+          <box size="0.22 0.26 0.006"/>
+        </geometry>
+        <material name="amr_badge_panel"/>
+      </visual>
+      <!-- 4. Identification Accent Trim -->
+      <visual name="id_badge_trim">
+        <origin xyz="0 0 ${chassis_height + 0.007}" rpy="0 0 0"/>
+        <geometry>
+          <box size="0.20 0.24 0.004"/>
+        </geometry>
+        <material name="amr_accent_cyan"/>
+      </visual>
+      <!-- 5. Identification Nameplate Face -->
+      <visual name="id_badge_face">
+        <origin xyz="0 0 ${chassis_height + 0.010}" rpy="0 0 0"/>
+        <geometry>
+          <box size="0.16 0.20 0.004"/>
+        </geometry>
+        <material name="amr_white_text"/>
+      </visual>
+      <!-- 6. Active Autonomous Status Indicator Ring (Rear Center Deck) -->
+      <visual name="status_beacon">
+        <origin xyz="${-chassis_length / 2.0 + 0.09} 0.0 ${chassis_height + 0.012}" rpy="0 0 0"/>
+        <geometry>
+          <cylinder radius="0.035" length="0.024"/>
+        </geometry>
+        <material name="amr_status_green"/>
+      </visual>
+      <!-- Exact collision box preserved from M1/M2 -->
+      <collision>
         <origin xyz="0 0 ${chassis_height / 2.0}" rpy="0 0 0"/>
         <geometry>
           <box size="${chassis_length} ${chassis_width} ${chassis_height}"/>
         </geometry>
-        <material name="amr_orange"/>
-      </visual>
-      <collision>
-        <origin xyz="0 0 ${chassis_height / 2.0}" rpy="0 0 0"/>
-        <geometry>
-          <box size="${chassis_length} ${chassis_width} ${chassis_height}"/>
-        </geometry>
-      </collision>
+      </collision>
+      <!-- Exact inertial parameters preserved from M1/M2 -->
       <inertial>
         <origin xyz="0 0 ${chassis_height / 2.0}" rpy="0 0 0"/>
@@ -56,17 +100,28 @@
     </joint>
     <link name="${prefix}left_wheel">
-      <visual>
-        <origin xyz="0 0 0" rpy="1.57079632679 0 0"/>
-        <geometry>
-          <cylinder radius="${wheel_radius}" length="${wheel_width}"/>
-        </geometry>
-        <material name="amr_black"/>
-      </visual>
-      <collision>
-        <origin xyz="0 0 0" rpy="1.57079632679 0 0"/>
-        <geometry>
-          <cylinder radius="${wheel_radius}" length="${wheel_width}"/>
-        </geometry>
-      </collision>
+      <!-- Rubber Tire Tread -->
+      <visual name="tire">
+        <origin xyz="0 0 0" rpy="1.57079632679 0 0"/>
+        <geometry>
+          <cylinder radius="${wheel_radius}" length="${wheel_width}"/>
+        </geometry>
+        <material name="amr_rubber_black"/>
+      </visual>
+      <!-- Silver Alloy Rim Hub -->
+      <visual name="rim">
+        <origin xyz="0 0 0" rpy="1.57079632679 0 0"/>
+        <geometry>
+          <cylinder radius="${wheel_radius * 0.62}" length="${wheel_width + 0.002}"/>
+        </geometry>
+        <material name="amr_rim_silver"/>
+      </visual>
+      <!-- Exact collision preserved -->
+      <collision>
+        <origin xyz="0 0 0" rpy="1.57079632679 0 0"/>
+        <geometry>
+          <cylinder radius="${wheel_radius}" length="${wheel_width}"/>
+        </geometry>
+      </collision>
+      <!-- Exact inertial preserved -->
       <inertial>
         <mass value="${wheel_mass}"/>
@@ -88,17 +143,28 @@
     </joint>
     <link name="${prefix}right_wheel">
-      <visual>
-        <origin xyz="0 0 0" rpy="1.57079632679 0 0"/>
-        <geometry>
-          <cylinder radius="${wheel_radius}" length="${wheel_width}"/>
-        </geometry>
-        <material name="amr_black"/>
-      </visual>
-      <collision>
-        <origin xyz="0 0 0" rpy="1.57079632679 0 0"/>
-        <geometry>
-          <cylinder radius="${wheel_radius}" length="${wheel_width}"/>
-        </geometry>
-      </collision>
+      <!-- Rubber Tire Tread -->
+      <visual name="tire">
+        <origin xyz="0 0 0" rpy="1.57079632679 0 0"/>
+        <geometry>
+          <cylinder radius="${wheel_radius}" length="${wheel_width}"/>
+        </geometry>
+        <material name="amr_rubber_black"/>
+      </visual>
+      <!-- Silver Alloy Rim Hub -->
+      <visual name="rim">
+        <origin xyz="0 0 0" rpy="1.57079632679 0 0"/>
+        <geometry>
+          <cylinder radius="${wheel_radius * 0.62}" length="${wheel_width + 0.002}"/>
+        </geometry>
+        <material name="amr_rim_silver"/>
+      </visual>
+      <!-- Exact collision preserved -->
+      <collision>
+        <origin xyz="0 0 0" rpy="1.57079632679 0 0"/>
+        <geometry>
+          <cylinder radius="${wheel_radius}" length="${wheel_width}"/>
+        </geometry>
+      </collision>
+      <!-- Exact inertial preserved -->
       <inertial>
         <mass value="${wheel_mass}"/>

File: src/amr_fleet_description/urdf/amr_lidar.xacro (robot description, xacro)
@@ -13,11 +13,29 @@
     </joint>
     <link name="${prefix}laser_frame">
-      <visual>
-        <origin xyz="0 0 0.02" rpy="0 0 0"/>
+      <!-- 1. Lower Turret Mount Base -->
+      <visual name="lidar_mount">
+        <origin xyz="0 0 0.010" rpy="0 0 0"/>
         <geometry>
-          <cylinder radius="0.04" length="0.04"/>
+          <cylinder radius="0.048" length="0.020"/>
         </geometry>
-        <material name="amr_blue"/>
+        <material name="amr_chassis_dark"/>
       </visual>
+      <!-- 2. Rotating Sensor Turret Body -->
+      <visual name="lidar_turret">
+        <origin xyz="0 0 0.028" rpy="0 0 0"/>
+        <geometry>
+          <cylinder radius="0.038" length="0.022"/>
+        </geometry>
+        <material name="amr_dark_grey"/>
+      </visual>
+      <!-- 3. Optical Sensor Window Aperture -->
+      <visual name="lidar_optical_window">
+        <origin xyz="0 0 0.028" rpy="0 0 0"/>
+        <geometry>
+          <cylinder radius="0.041" length="0.010"/>
+        </geometry>
+        <material name="amr_sensor_lens"/>
+      </visual>
+      <!-- Exact collision geometry preserved from M1/M2 -->
       <collision>
         <origin xyz="0 0 0.02" rpy="0 0 0"/>
@@ -26,4 +44,5 @@
         </geometry>
       </collision>
+      <!-- Exact inertial parameters preserved from M1/M2 -->
       <inertial>
         <origin xyz="0 0 0.02" rpy="0 0 0"/>

File: src/amr_fleet_description/urdf/amr_materials.xacro (robot description, xacro)
@@ -1,4 +1,5 @@
 <?xml version="1.0"?>
 <robot xmlns:xacro="http://www.ros.org/wiki/xacro">
+  <!-- Classic Palette (Preserved for compatibility) -->
   <material name="amr_orange">
     <color rgba="0.95 0.45 0.1 1.0"/>
@@ -16,3 +17,34 @@
     <color rgba="0.1 0.5 0.9 1.0"/>
   </material>
+  <!-- M2.5 Polished Industrial Palette -->
+  <material name="amr_chassis_dark">
+    <color rgba="0.12 0.14 0.16 1.0"/>
+  </material>
+  <material name="amr_safety_orange">
+    <color rgba="0.90 0.36 0.00 1.0"/>
+  </material>
+  <material name="amr_rim_silver">
+    <color rgba="0.65 0.69 0.72 1.0"/>
+  </material>
+  <material name="amr_rubber_black">
+    <color rgba="0.08 0.09 0.10 1.0"/>
+  </material>
+  <material name="amr_sensor_lens">
+    <color rgba="0.10 0.12 0.17 1.0"/>
+  </material>
+  <material name="amr_status_green">
+    <color rgba="0.00 0.90 0.46 1.0"/>
+  </material>
+  <material name="amr_status_amber">
+    <color rgba="1.00 0.60 0.00 1.0"/>
+  </material>
+  <material name="amr_badge_panel">
+    <color rgba="0.05 0.07 0.09 1.0"/>
+  </material>
+  <material name="amr_accent_cyan">
+    <color rgba="0.00 0.74 0.83 1.0"/>
+  </material>
+  <material name="amr_white_text">
+    <color rgba="0.96 0.96 0.98 1.0"/>
+  </material>
 </robot>
